File: backup/percobaan.kicad_pcb (KiCad board)
At the start: 2 copper layers, 134.5 x 87 mm, 11 parts, among them J1 soil moist, J2 Screw_Terminal_01x04, U1 LM393

Commit message: Add files via upload
Parts:
- moved J1 6.74 mm to (53.8, 83.2), turned to -90 degrees
Routing:
- net GND: track 457.6 -> 472.7 mm
- net VCC: track 361.8 -> 352.2 mm
- added copper zone on B.Cu, net (none)
- removed copper zone on B.Cu, net GND
